File: eagle/pinoccio.brd (EAGLE design)
At the start: 25.4 x 50.8 mm, 51 parts, among them Q1 16MHz, Q2 32.768k, Q4 MOSFET-PCHANNEL, Q5 TRANSISTOR-NPN-DUAL, U1 MCP73831, U2 3.3V, U4 ATMEGA128RFA1, X1 USB-MICROB, Y2 ANTENNA2SMD5

Commit message: Updated pinoccio copper/mask logo
Parts:
- removed U$6: (no value), Pinoccio:LOGO-OSHW-SS
- moved U$2 0.72 mm to (17.6, 47.3)
- moved U$3 0.70 mm to (17.6, 47.3)
- moved R4 0.10 mm to (10.3, 38.1)
- moved R3 0.05 mm to (10.6, 44.0)
Routing:
- net GND: vias 82 -> 83
Other:
- board text removed: "/Volumes/Data/Users/eric/Desktop/Untitled-1.bmp"
Changed lines of the file:
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@@
 <layer number="20" name="Dimension" color="6" fill="1" visible="yes" active="yes"/>
 <layer number="21" name="tPlace" color="16" fill="1" visible="yes" active="yes"/>
-<layer number="22" name="bPlace" color="14" fill="1" visible="no" active="yes"/>
+<layer number="22" name="bPlace" color="14" fill="1" visible="yes" active="yes"/>
 <layer number="23" name="tOrigins" color="15" fill="1" visible="yes" active="yes"/>
 <layer number="24" name="bOrigins" color="15" fill="1" visible="yes" active="yes"/>
@@
 <layer number="39" name="tKeepout" color="4" fill="11" visible="no" active="yes"/>
 <layer number="40" name="bKeepout" color="1" fill="11" visible="yes" active="yes"/>
-<layer number="41" name="tRestrict" color="4" fill="10" visible="yes" active="yes"/>
+<layer number="41" name="tRestrict" color="4" fill="10" visible="no" active="yes"/>
 <layer number="42" name="bRestrict" color="1" fill="10" visible="yes" active="yes"/>
 <layer number="43" name="vRestrict" color="2" fill="10" visible="no" active="yes"/>
@@
 <rectangle x1="12.92" y1="7.42" x2="13.48" y2="10.64" layer="1"/>
 <text x="-10.4648" y="-10.2362" size="1.27" layer="51" font="vector" ratio="15">Licensed under CERN OHL v.1.1</text>
-<text x="0" y="-0.0635" size="0.0254" layer="29" font="vector">/Volumes/Data/Users/eric/Desktop/Untitled-1.bmp</text>
+<rectangle x1="14.7828" y1="47.9552" x2="15.3162" y2="48.768" layer="42"/>
 </plain>
 <attributes>
@@
 <element name="C5" library="SparkFun" package="0402-CAP" value="4.7uF" x="11.1506" y="41.7322" smashed="yes" rot="R270"/>
 <element name="D2" library="SparkFun" package="LED-0603" value="Yellow" x="12.7" y="43.8658" smashed="yes" rot="R90"/>
-<element name="R3" library="SparkFun" package="0402-RES" value="470" x="10.6426" y="43.942" smashed="yes" rot="R90"/>
+<element name="R3" library="SparkFun" package="0402-RES" value="470" x="10.6426" y="43.9928" smashed="yes" rot="R90"/>
 <element name="X1" library="SparkFun" package="USB-MICROB" value="USB-MICROB" x="12.7" y="48.6664" locked="yes" smashed="yes" rot="R180">
 <attribute name="VALUE" x="16.51" y="48.6664" size="0.4064" layer="27" rot="R180"/>
@@
 <attribute name="VALUE" x="9.7155" y="41.0845" size="0.4064" layer="27" rot="R180"/>
 </element>
-<element name="R4" library="SparkFun" package="0402-RES" value="2K" x="10.287" y="38.227" smashed="yes">
-<attribute name="VALUE" x="9.271" y="37.084" size="0.4064" layer="27" font="vector"/>
+<element name="R4" library="SparkFun" package="0402-RES" value="2K" x="10.3124" y="38.1254" smashed="yes">
+<attribute name="VALUE" x="9.2964" y="36.9824" size="0.4064" layer="27" font="vector"/>
 </element>
 <element name="U4" library="Pinoccio" package="QFN-64" value="ATMEGA128RFA1" x="12.7" y="18.2118" smashed="yes" rot="R90">
@@
 <attribute name="VALUE" x="18.726" y="38.8632" size="1.27" layer="27" rot="R180"/>
 </element>
-<element name="U$2" library="Pinoccio" package="LOGO-PINOCCIO-COPPER" value="" x="18.1356" y="46.8122" rot="MR0"/>
-<element name="U$3" library="Pinoccio" package="LOGO-PINOCCIO-STOP" value="" x="18.1356" y="46.8122" rot="MR0"/>
-<element name="U$6" library="Pinoccio" package="LOGO-OSHW-SS" value="" x="14.0716" y="41.0718" rot="MR0"/>
+<element name="U$2" library="Pinoccio" package="LOGO-PINOCCIO-COPPER" value="" x="17.6022" y="47.2948" rot="MR0"/>
+<element name="U$3" library="Pinoccio" package="LOGO-PINOCCIO-STOP" value="" x="17.6276" y="47.2948" rot="MR0"/>
 </elements>
 <signals>
@@
 <wire x1="3.7338" y1="44.7294" x2="4.8266" y2="43.5858" width="0.508" layer="1"/>
 <wire x1="4.8266" y1="43.5858" x2="5.8684" y2="43.535" width="0.508" layer="1"/>
-<wire x1="6.3246" y1="45.3898" x2="10.795" y2="45.3898" width="0.508" layer="1"/>
-<wire x1="10.795" y1="45.3898" x2="11.4" y2="45.9948" width="0.508" layer="1"/>
+<wire x1="6.3246" y1="45.4152" x2="10.795" y2="45.4152" width="0.508" layer="1"/>
+<wire x1="10.795" y1="45.4152" x2="11.4" y2="45.9948" width="0.508" layer="1"/>
 <wire x1="11.4" y1="45.9948" x2="11.4" y2="46.0164" width="0.508" layer="1"/>
-<wire x1="6.3246" y1="45.3898" x2="5.715" y2="44.7802" width="0.508" layer="1"/>
-<wire x1="5.715" y1="44.7802" x2="5.715" y2="43.688" width="0.508" layer="1"/>
+<wire x1="6.3246" y1="45.4152" x2="5.715" y2="44.8056" width="0.508" layer="1"/>
+<wire x1="5.715" y1="44.8056" x2="5.715" y2="43.688" width="0.508" layer="1"/>
 <wire x1="5.715" y1="43.688" x2="5.842" y2="43.561" width="0.508" layer="1"/>
 <wire x1="5.8684" y1="43.535" x2="5.8668" y2="43.5858" width="0.508" layer="1"/>
@@
 <via x="16.5918" y="35.737" extent="1-16" drill="0.3302"/>
 <via x="18.4206" y="35.737" extent="1-16" drill="0.3302"/>
-<via x="5.2634" y="36.3212" extent="1-16" drill="0.3302"/>
+<via x="5.4158" y="36.3212" extent="1-16" drill="0.3302"/>
 <via x="19.6164" y="10.16" extent="1-16" drill="0.3302"/>
 <via x="16.7068" y="10.16" extent="1-16" drill="0.3302"/>
@@
 <via x="9.8862" y="45.7192" extent="1-16" drill="0.3302"/>
 <via x="8.794" y="45.7192" extent="1-16" drill="0.3302"/>
-<wire x1="10.937" y1="38.227" x2="11.049" y2="38.442" width="0.2032" layer="1"/>
+<wire x1="10.9624" y1="38.1254" x2="11.049" y2="38.442" width="0.2032" layer="1"/>
 <wire x1="11.049" y1="38.442" x2="11.049" y2="40.1828" width="0.2032" layer="1"/>
 <via x="6.7112" y="45.7192" extent="1-16" drill="0.3302"/>
@@
 <via x="15.2336" y="10.16" extent="1-16" drill="0.3302"/>
 <via x="4.505" y="14.4518" extent="1-16" drill="0.3302"/>
-<via x="10.922" y="20.4216" extent="1-16" drill="0.3302" alwaysstop="yes"/>
-<via x="10.922" y="19.2278" extent="1-16" drill="0.3302" alwaysstop="yes"/>
-<via x="10.922" y="18.034" extent="1-16" drill="0.3302" alwaysstop="yes"/>
-<via x="12.7" y="19.2278" extent="1-16" drill="0.3302" alwaysstop="yes"/>
-<via x="12.7" y="20.4216" extent="1-16" drill="0.3302" alwaysstop="yes"/>
-<via x="14.478" y="20.4216" extent="1-16" drill="0.3302" alwaysstop="yes"/>
-<via x="14.478" y="19.2278" extent="1-16" drill="0.3302" alwaysstop="yes"/>
+<via x="10.922" y="20.4216" extent="1-16" drill="0.3302"/>
+<via x="10.922" y="19.2278" extent="1-16" drill="0.3302"/>
+<via x="10.922" y="18.034" extent="1-16" drill="0.3302"/>
+<via x="12.7" y="19.2278" extent="1-16" drill="0.3302"/>
+<via x="12.7" y="20.4216" extent="1-16" drill="0.3302"/>
+<via x="14.478" y="20.4216" extent="1-16" drill="0.3302"/>
+<via x="14.478" y="19.2278" extent="1-16" drill="0.3302"/>
 <via x="17.6784" y="27.051" extent="1-16" drill="0.3302"/>
 <via x="17.3482" y="27.9654" extent="1-16" drill="0.3302"/>
@@
 <via x="24.2316" y="49.5046" extent="1-16" drill="0.3302"/>
 <via x="24.2316" y="44.1444" extent="1-16" drill="0.3302"/>
-<via x="5.619" y="46.2788" extent="1-16" drill="0.3302"/>
+<via x="5.5428" y="46.1264" extent="1-16" drill="0.3302"/>
 <via x="2.7742" y="49.5046" extent="1-16" drill="0.3302"/>
 <via x="4.7808" y="49.5046" extent="1-16" drill="0.3302"/>
-<via x="0.9962" y="46.2788" extent="1-16" drill="0.3302"/>
-<via x="5.4412" y="34.3654" extent="1-16" drill="0.3302"/>
+<via x="1.4534" y="46.5074" extent="1-16" drill="0.3302"/>
+<via x="5.4412" y="34.4162" extent="1-16" drill="0.3302"/>
+<via x="7.0668" y="49.5046" extent="1-16" drill="0.3302"/>
 </signal>
 <signal name="VCC" class="1">
@@
 <contactref element="R4" pad="1"/>
 <wire x1="9.6148" y1="39.4957" x2="9.713" y2="39.5939" width="0.2032" layer="1"/>
-<wire x1="9.637" y1="38.227" x2="9.713" y2="38.227" width="0.4064" layer="1"/>
+<wire x1="9.6624" y1="38.1254" x2="9.713" y2="38.227" width="0.4064" layer="1"/>
 <wire x1="9.713" y1="38.227" x2="9.713" y2="39.5939" width="0.4064" layer="1"/>
 </signal>
@@
 <via x="9.6774" y="43.7642" extent="1-16" drill="0.3302"/>
 <wire x1="3.9116" y1="41.5925" x2="3.9116" y2="32.6136" width="0.2032" layer="16"/>
-<wire x1="10.6426" y1="43.292" x2="10.2004" y2="43.7746" width="0.2032" layer="1"/>
-<wire x1="10.2004" y1="43.7746" x2="9.6774" y2="43.7642" width="0.2032" layer="1"/>
 <wire x1="9.8194" y1="42.3005" x2="9.713" y2="42.1941" width="0.2032" layer="1"/>
 <wire x1="9.8194" y1="42.3005" x2="9.8194" y2="43.6222" width="0.2032" layer="1"/>
@@
 <wire x1="6.4008" y1="32.131" x2="6.0706" y2="31.7754" width="0.2032" layer="16"/>
 <wire x1="6.0706" y1="31.7754" x2="4.7498" y2="31.7754" width="0.2032" layer="16"/>
+<wire x1="9.6774" y1="43.7642" x2="10.0988" y2="43.3428" width="0.2032" layer="1"/>
+<wire x1="10.0988" y1="43.3428" x2="10.6426" y2="43.3428" width="0.2032" layer="1"/>
 </signal>
 <signal name="N$46">
@@
 <contactref element="D2" pad="C"/>
 <contactref element="R3" pad="2"/>
-<wire x1="11.95" y1="43.8658" x2="11.3688" y2="43.8658" width="0.2032" layer="1"/>
-<wire x1="11.3688" y1="43.8658" x2="10.6426" y2="44.592" width="0.2032" layer="1"/>
+<wire x1="11.95" y1="43.8658" x2="11.173" y2="44.6428" width="0.2032" layer="1"/>
+<wire x1="11.173" y1="44.6428" x2="10.6426" y2="44.6428" width="0.2032" layer="1"/>
 </signal>
 <signal name="N$3">
