File: eagle/pinoccio.sch (EAGLE design)
At the start: 69 parts, among them IC1 ATMEGA16U2QFN32, J1 AVR_SPI_PRG_6, Q1 16MHz, Q2 32.768k, Q3 16MHz, Q4 MOSFET-PCHANNELSMD, U1 MCP73832, U2 TPS78233, U4 ATMEGA128RFA1, X1 USB-MICROB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

Commit message: version 0.11 updates
Parts:
- removed C1: 100nF, Pinoccio:CAP0402-CAP
Connections:
- removed net VBAT-AS: C6.1, JP-R.3, JP1.2, S2.P, U2.EN, U2.IN
- new net VIN: C6.1, JP1.2, S2.P, U2.EN, U2.IN
- net AREF: no longer C1.1
- net GND: no longer C1.2
- net VBAT: now also JP-R.3
Other:
- note added: "0.11"
- note removed: "0.10"
Changed lines of the file:
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@@
 <part name="GND6" library="SparkFun" deviceset="GND" device=""/>
 <part name="GND8" library="SparkFun" deviceset="GND" device=""/>
-<part name="C1" library="Pinoccio" deviceset="CAP" device="0402-CAP" value="100nF"/>
-<part name="GND13" library="SparkFun" deviceset="GND" device=""/>
 <part name="R6" library="Pinoccio" deviceset="RESISTOR" device="0402-RES" value="470"/>
 <part name="R20" library="Pinoccio" deviceset="RESISTOR" device="0402-RES" value="10k"/>
@@
 <sheet>
 <plain>
-<text x="238.76" y="1.27" size="2.54" layer="94" font="vector">0.10</text>
+<text x="238.76" y="1.27" size="2.54" layer="94" font="vector">0.11</text>
 <rectangle x1="0.38735" y1="0.29845" x2="0.41275" y2="0.31115" layer="21"/>
 <rectangle x1="0.36195" y1="0.31115" x2="0.45085" y2="0.32385" layer="21"/>
@@
 <instance part="GND6" gate="1" x="15.24" y="96.52"/>
 <instance part="GND8" gate="1" x="5.08" y="83.82"/>
-<instance part="C1" gate="G$1" x="121.92" y="149.86" smashed="yes">
-<attribute name="NAME" x="115.824" y="150.241" size="1.778" layer="95"/>
-<attribute name="VALUE" x="123.444" y="147.701" size="1.778" layer="96"/>
-</instance>
-<instance part="GND13" gate="1" x="121.92" y="144.78"/>
 <instance part="R6" gate="G$1" x="96.52" y="124.46" rot="MR90"/>
 <instance part="R20" gate="G$1" x="10.16" y="48.26" rot="R270"/>
@@
 </segment>
 <segment>
-<pinref part="C1" gate="G$1" pin="2"/>
-<pinref part="GND13" gate="1" pin="GND"/>
-</segment>
-<segment>
 <pinref part="R20" gate="G$1" pin="2"/>
 <pinref part="GND17" gate="1" pin="GND"/>
@@
 <segment>
 <pinref part="U4" gate="G$1" pin="AREF"/>
-<wire x1="144.78" y1="157.48" x2="121.92" y2="157.48" width="0.1524" layer="91"/>
-<wire x1="121.92" y1="157.48" x2="121.92" y2="154.94" width="0.1524" layer="91"/>
-<label x="114.3" y="154.94" size="1.778" layer="95"/>
-<pinref part="C1" gate="G$1" pin="1"/>
-<wire x1="121.92" y1="157.48" x2="114.3" y2="157.48" width="0.1524" layer="91"/>
-<junction x="121.92" y="157.48"/>
+<wire x1="144.78" y1="157.48" x2="132.08" y2="157.48" width="0.1524" layer="91"/>
+<label x="132.08" y="157.48" size="1.778" layer="95"/>
 </segment>
 <segment>
@@
 <label x="190.5" y="35.56" size="1.778" layer="95"/>
 </segment>
+<segment>
+<pinref part="JP-R" gate="G$1" pin="3"/>
+<wire x1="236.22" y1="119.38" x2="223.52" y2="119.38" width="0.1524" layer="91"/>
+<label x="223.52" y="119.38" size="1.778" layer="95"/>
+</segment>
 </net>
-<net name="VBAT-AS" class="0">
+<net name="VIN" class="0">
 <segment>
 <wire x1="30.48" y1="68.58" x2="33.02" y2="68.58" width="0.1524" layer="91"/>
@@
 <junction x="33.02" y="68.58"/>
 </segment>
-<segment>
-<pinref part="JP-R" gate="G$1" pin="3"/>
-<wire x1="236.22" y1="119.38" x2="223.52" y2="119.38" width="0.1524" layer="91"/>
-<label x="223.52" y="119.38" size="1.778" layer="95"/>
-</segment>
 </net>
